Commit message: CALLING ON OLD CODE IN URDF. FIXED THIS LINE IN X500_DESC.

File: x500_description/urdf/holybro_drone_gz_assembly.urdf (robot description, URDF)
Before this commit: robot holybro_drone_assembly, 3 links, 2 joints
Links:
- added link base_footprint
Joints:
- added joint base_joint: type fixed, parent base_footprint, child base_link, origin xyz=0 0 -0.21528 rpy=3.14 0 0

Commit message: Setup for relative aruco marker measurement based off NED Body_link (Written as base link in URDF code). This version of the OFFBOARD code is the most consistent with landing and has minimal errors.

File: x500_description/urdf/holybro_drone_gz_assembly.urdf (robot description, URDF)
Before this commit: robot holybro_drone_assembly, 4 links, 3 joints
Links:
- added link base_link_NED
Joints:
- added joint body_link_NED: type fixed, parent base_link_NED, child base_link, origin xyz=0 0 -0.0398999999999999 rpy=3.14 0 0
- joint base_joint: child base_link -> base_link_NED; origin xyz=0 0 -0.21528 rpy=3.14 0 0 -> xyz=0 0 -0.21528 rpy=0 0 0
