Commit message: Update file paths to X500_description not drone_urdf

File: x500_description/urdf/holybro_drone_assembly.urdf (robot description, URDF)
Before this commit: robot holybro_drone_assembly, 3 links, 2 joints
Links:
- added link base_footprint
- link base_link: geometry collision mesh filename=package://x500_description/meshes/visual/base_link.STL; visual mesh filename=package://x500_description/meshes/visual/base_link.STL
- link body_link: geometry collision mesh filename=package://x500_description/meshes/visual/body_link.STL; visual mesh filename=package://x500_description/meshes/visual/body_link.STL
- link camera_link: geometry collision mesh filename=package://x500_description/meshes/visual/camera_link.STL; visual mesh filename=package://x500_description/meshes/visual/camera_link.STL
Joints:
- added joint base_joint: type fixed, parent base_footprint, child base_link, origin xyz=0 0 -0.21528 rpy=3.14 0 0

File: x500_description/urdf/holybro_drone_gz_assembly.urdf (robot description, URDF)
Before this commit: robot holybro_drone_assembly, 4 links, 3 joints
Links:
- link base_link: geometry collision mesh filename=package://x500_description/meshes/visual/base_link.STL; visual mesh filename=package://x500_description/meshes/visual/base_link.STL
- link body_link: geometry collision mesh filename=package://x500_description/meshes/visual/body_link.STL; visual mesh filename=package://x500_description/meshes/visual/body_link.STL
- link camera_link: geometry collision mesh filename=package://x500_description/meshes/visual/camera_link.STL; visual mesh filename=package://x500_description/meshes/visual/camera_link.STL

Commit message: Updated URDF. Important Changes done to the setup.py and urdf files. When updating URDF, launch file creation/links broke... in addition to odd ros2 errors (not releated)

File: x500_description/urdf/holybro_drone_assembly.urdf (robot description, URDF)
Before this commit: robot holybro_drone_assembly, 4 links, 3 joints
Links:
- added link base_ned_link, mass 0.003562; collision mesh filename=package://x500_description/meshes/visual/base_ned_link.STL; visual mesh filename=package://x500_description/meshes/visual/base_ned_link.STL
- link base_footprint: mass None -> 0.13605; geometry collision mesh filename=package://x500_description/meshes/visual/base_footprint.STL; visual mesh filename=package://x500_description/meshes/visual/base_footprint.STL
- link base_link: mass None -> 0.455776613743598
- link body_link: mass 0.453039078577497 -> 0.69044
- link camera_link: mass 0.0925592950450192 -> 0.11461
Joints:
- removed joint body_link
- removed joint camera_link
- added joint base_footprint_joint: type fixed, parent base_footprint, child base_link, origin xyz=0 0 0.001 rpy=0 0 0
- added joint base_ned_joint: type fixed, parent base_link, child base_ned_link, origin xyz=0 0 0 rpy=-3.14159265358979 0 0, axis 0 0 0
- added joint body_joint: type fixed, parent base_link, child body_link, origin xyz=0 0 0.0461 rpy=0 0 0, axis 0 0 0
- added joint camera_joint: type fixed, parent base_link, child camera_link, origin xyz=0.1272 0 -0.0465999999999999 rpy=3.14159265358979 0 -1.5707963267949, axis 0 0 0
- joint base_joint: axis (none) -> 0 0 0; origin xyz=0 0 -0.21528 rpy=3.14 0 0 -> xyz=0 0 -0.216276433489377 rpy=3.14159265358979 0 0

File: x500_description/urdf/holybro_drone_gz_assembly.urdf (robot description, URDF)
Before this commit: robot holybro_drone_assembly, 5 links, 4 joints
Links:
- removed link base_link_NED
- added link base_ned_link, mass 0.003562; collision mesh filename=package://x500_description/meshes/visual/base_ned_link.STL; visual mesh filename=package://x500_description/meshes/visual/base_ned_link.STL
- link base_footprint: mass None -> 0.13605; geometry collision mesh filename=package://x500_description/meshes/visual/base_footprint.STL; visual mesh filename=package://x500_description/meshes/visual/base_footprint.STL
- link base_link: mass None -> 0.455776613743598
- link body_link: mass 0.453039078577497 -> 0.69044
- link camera_link: mass 0.0925592950450192 -> 0.11461
Joints:
- removed joint body_link
- removed joint body_link_NED
- removed joint camera_link
- added joint base_ned_joint: type fixed, parent base_link, child base_ned_link, origin xyz=0 0 0 rpy=-3.14159265358979 0 0, axis 0 0 0
- added joint body_joint: type fixed, parent base_link, child body_link, origin xyz=0 0 0.0461 rpy=0 0 0, axis 0 0 0
- added joint camera_joint: type fixed, parent base_link, child camera_link, origin xyz=0.1272 0 -0.0465999999999999 rpy=3.14159265358979 0 -1.5707963267949, axis 0 0 0
- joint base_joint: axis (none) -> 0 0 0; child base_link_NED -> base_link; origin xyz=0 0 -0.21528 rpy=0 0 0 -> xyz=0 0 -0.216276433489377 rpy=3.14159265358979 0 0

Commit message: Backing up Jetson development

File: x500_description/urdf/holybro_drone_assembly.urdf (robot description, URDF)
Before this commit: robot holybro_drone_assembly, 4 links, 3 joints
Links:
- added link base_ned_link, mass 0.003562; collision mesh filename=package://x500_description/meshes/visual/base_ned_link.STL; visual mesh filename=package://x500_description/meshes/visual/base_ned_link.STL
- link base_footprint: mass None -> 0.13605; geometry collision mesh filename=package://x500_description/meshes/visual/base_footprint.STL; visual mesh filename=package://x500_description/meshes/visual/base_footprint.STL
- link base_link: mass None -> 0.455776613743598
- link body_link: mass 0.453039078577497 -> 0.69044
- link camera_link: mass 0.0925592950450192 -> 0.11461
Joints:
- removed joint body_link
- removed joint camera_link
- added joint base_ned_joint: type fixed, parent base_link, child base_ned_link, origin xyz=0 0 0 rpy=-3.14159265358979 0 0, axis 0 0 0
- added joint body_joint: type fixed, parent base_link, child body_link, origin xyz=0 0 0.0461 rpy=0 0 0, axis 0 0 0
- added joint camera_joint: type fixed, parent base_link, child camera_link, origin xyz=0.1272 0 -0.0465999999999999 rpy=3.14159265358979 0 -1.5707963267949, axis 0 0 0
- joint base_joint: axis (none) -> 0 0 0; origin xyz=0 0 -0.21528 rpy=3.14 0 0 -> xyz=0 0 -0.216276433489377 rpy=3.14159265358979 0 0

Commit message: Working code prepared for CCTOMM 2025. See jetson branch for this commit with the updated parts of code as files were switched arond often during testing.

File: x500_description/urdf/holybro_drone_assembly.urdf (robot description, URDF)
Before this commit: robot holybro_drone_assembly, 5 links, 5 joints
Links:
- link base_footprint: mass 0.13605 -> 0.296919523990479
- link base_link: mass 0.455776613743598 -> 0.0752275868088825
- link base_ned_link: mass 0.003562 -> 0.00437682945739925
- link body_link: mass 0.69044 -> 16.5303129418879
- link camera_link: mass 0.11461 -> 0.0727080976862257
Joints:
- removed joint base_footprint_joint
- joint base_joint: origin xyz=0 0 -0.216276433489377 rpy=3.14159265358979 0 0 -> xyz=0 0 -0.137 rpy=-3.14159265358979 0 0
- joint base_ned_joint: origin xyz=0 0 0 rpy=-3.14159265358979 0 0 -> xyz=0 0 0 rpy=3.14159265358979 0 0
- joint camera_joint: origin xyz=0.1272 0 -0.0465999999999999 rpy=3.14159265358979 0 -1.5707963267949 -> xyz=0.07546095994 0 -0.0330999999999999 rpy=3.14159265358979 0 -1.57079632679489

File: x500_description/urdf/holybro_drone_gz_assembly.urdf (robot description, URDF)
Before this commit: robot holybro_drone_assembly, 5 links, 4 joints
Links:
- link base_footprint: mass 0.13605 -> 0.296919523990479
- link base_link: mass 0.455776613743598 -> 0.0752275868088825
- link base_ned_link: mass 0.003562 -> 0.00437682945739925
- link body_link: mass 0.69044 -> 16.5303129418879
- link camera_link: mass 0.11461 -> 0.0727080976862257
Joints:
- joint base_joint: origin xyz=0 0 -0.216276433489377 rpy=3.14159265358979 0 0 -> xyz=0 0 -0.137 rpy=-3.14159265358979 0 0
- joint base_ned_joint: origin xyz=0 0 0 rpy=-3.14159265358979 0 0 -> xyz=0 0 0 rpy=3.14159265358979 0 0
- joint camera_joint: origin xyz=0.1272 0 -0.0465999999999999 rpy=3.14159265358979 0 -1.5707963267949 -> xyz=0.07546095994 0 -0.0330999999999999 rpy=3.14159265358979 0 -1.57079632679489
